Commit message: Cleanup

File: urdf/scara.urdf (robot description, URDF)
Before this commit: robot scara, 5 links, 4 joints
Joints:
- removed joint link1_to_base
- removed joint link2_to_link1
- added joint base_to_link1: type revolute, parent base_link, child link_1, origin xyz=0 0 0.4, axis 0 0 1, limit lower=-2.5 upper=2.5 effort=300 velocity=0.1
- added joint link1_to_link2: type revolute, parent link_1, child link_2, origin xyz=0.3 0 0, axis 0 0 1, limit lower=-2.0 upper=2.0 effort=300 velocity=0.1
